File: Buck Convertor (12V 6A).kicad_sch (KiCad schematic)
At the start: 41 parts, among them J1 1726480102, J2 1726480102, J3 Conn_01x03, J4 Conn_01x03, Q1 2N7002, Q2 NTD2955T4G, U1 SIC438BED-T1-GE3

Commit message: Fixed PFET being wrong size
Parts:
- removed Q2: NTD2955T4G, xavier6a_12v:DPAK-369C_ONS, symbol Simulation_SPICE:PMOS
- added Q2: NTD2955T4G, Buck12V6A:TO-252-2_L6.6-W6.1-P4.57-LS9.9-TL-CW, symbol Buck12V6A:NTD2955T4G
- C1, C10: symbol xavier6a_12v:0805,100nF -> Buck12V6A:0805,100nF
- C12, C2, C3, C4, C5, C6, C7: symbol JLCPCB-Capacitors:0805,22uF -> Buck12V6A:0805,22uF
- C8: symbol xavier6a_12v:0805,4.7uF -> Buck12V6A:0805,4.7uF
- C9: symbol xavier6a_12v:0805,1uF -> Buck12V6A:0805,1uF
- CON1, CON2: symbol xavier6a_12v:6_Gold_Finger -> Buck12V6A:6_Gold_Finger
- D1: symbol xavier6a_12v:LED,0805,Yellow -> Buck12V6A:LED,0805,Yellow
- D3: symbol JLCPCB-Diodes:General,S10JC -> Buck12V6A:General,S10JC
- D4: footprint JLCPCB-Kicad-Footprints:D_SOD-323 -> Buck12V6A:D_SOD-323; symbol JLCPCB-Diodes:Zener,BZT52C16S -> Buck12V6A:Zener,BZT52C16S
- F1: footprint 3557_2:FUSE_3557-2 -> Buck12V6A:FUSE_3557-2; symbol 3557-2:3557-2 -> Buck12V6A:3557-2
- J1, J2: footprint 1726480102:CONN_SD-172648-0000_02_MOL -> Buck12V6A:CONN_SD-172648-0000_02_MOL; symbol xavier6a_12v:1726480102 -> Buck12V6A:1726480102; now not fitted
- J3, J4: symbol Connector_Generic:Conn_01x03 -> Buck12V6A:Conn_01x03; now not fitted; now left out of the parts list
- L1: footprint xavier6a_12v:ZEMS1040 -> Buck12V6A:ZEMS1040; symbol xavier6a_12v:ZE_ZEMS1040-3R3M -> Buck12V6A:ZE_ZEMS1040-3R3M
- Q1: symbol xavier6a_12v:2N7002 -> Buck12V6A:2N7002
- R1, R3: symbol xavier6a_12v:0805,1kΩ -> Buck12V6A:0805,1kΩ
- R10, R8: symbol Device:R -> Buck12V6A:R
- R11: symbol JLCPCB-Resistors:0805,51kΩ -> Buck12V6A:0805,51kΩ
- R12: symbol JLCPCB-Resistors:0805,510kΩ -> Buck12V6A:0805,510kΩ
- R13: symbol JLCPCB-Resistors:0805,300kΩ -> Buck12V6A:0805,300kΩ
- R2: symbol xavier6a_12v:0805,100Ω -> Buck12V6A:0805,100Ω
- R4, R9: symbol xavier6a_12v:0805,10kΩ -> Buck12V6A:0805,10kΩ
- R5: symbol xavier6a_12v:0805,2.2Ω -> Buck12V6A:0805,2.2Ω
- R6, R7: symbol xavier6a_12v:0805,200kΩ -> Buck12V6A:0805,200kΩ
- TP1, TP2, TP3: symbol dk_Test-Points:RCT-0C -> Buck12V6A:RCT-0C
- U1: footprint QFN_ED-T1-GE3_VIS -> Buck12V6A:QFN_ED-T1-GE3_VIS; symbol xavier6a_12v:SIC438BED-T1-GE3 -> Buck12V6A:SIC438BED-T1-GE3
Connections:
- net VINRAW: now also Q2.2 (D)
- net at D4.2, R3.1: now also Q2.1 (G)
- net at D4.1, F1.1_1: now also Q2.3 (S)
